File: Flight-controller-sch.sch (KiCad schematic (older format))
At the start: 0 parts

Commit message: Add headers for teensy
Parts:
- added P1, P3: CONN_01X14, symbol CONN_01X14
- added P2: CONN_01X03, symbol CONN_01X03
- added P4: CONN_01X05, symbol CONN_01X05
Other:
- note added: "Teensy 3.2\nconnection"
Changed lines of the file:
@@
 $EndSheet
 $Comp
-L PWR_FLAG #FLG?
+L PWR_FLAG #FLG01
 U 1 1 57476373
 P 1000 1000
-F 0 "#FLG?" H 1000 1095 50  0001 C CNN
+F 0 "#FLG01" H 1000 1095 50  0001 C CNN
 F 1 "PWR_FLAG" V 900 1000 50  0000 C CNN
 F 2 "" H 1000 1000 50  0000 C CNN
@@
 $EndComp
 $Comp
-L PWR_FLAG #FLG?
+L PWR_FLAG #FLG02
 U 1 1 5747639D
 P 1250 1000
-F 0 "#FLG?" H 1250 1095 50  0001 C CNN
+F 0 "#FLG02" H 1250 1095 50  0001 C CNN
 F 1 "PWR_FLAG" V 1150 1000 50  0000 C CNN
 F 2 "" H 1250 1000 50  0000 C CNN
@@
 $EndComp
 $Comp
-L GND #PWR?
+L GND #PWR03
 U 1 1 574763FE
 P 1250 1150
-F 0 "#PWR?" H 1250 900 50  0001 C CNN
+F 0 "#PWR03" H 1250 900 50  0001 C CNN
 F 1 "GND" H 1250 1000 50  0000 C CNN
 F 2 "" H 1250 1150 50  0000 C CNN
@@
 $EndComp
 $Comp
-L +12V #PWR?
+L +12V #PWR04
 U 1 1 5747642A
 P 1000 1150
-F 0 "#PWR?" H 1000 1000 50  0001 C CNN
+F 0 "#PWR04" H 1000 1000 50  0001 C CNN
 F 1 "+12V" H 1000 1290 50  0000 C CNN
 F 2 "" H 1000 1150 50  0000 C CNN
@@
 Battery IN
 $Comp
-L +12V #PWR?
+L +12V #PWR05
 U 1 1 57476580
 P 2000 1100
-F 0 "#PWR?" H 2000 950 50  0001 C CNN
+F 0 "#PWR05" H 2000 950 50  0001 C CNN
 F 1 "+12V" H 2000 1240 50  0000 C CNN
 F 2 "" H 2000 1100 50  0000 C CNN
@@
 Wire Wire Line
 	2000 1250 2500 1250
+$Comp
+L CONN_01X14 P1
+U 1 1 574781C0
+P 8800 5050
+F 0 "P1" H 8800 5800 50  0000 C CNN
+F 1 "CONN_01X14" V 8900 5050 50  0000 C CNN
+F 2 "" H 8800 5050 50  0000 C CNN
+F 3 "" H 8800 5050 50  0000 C CNN
+	1    8800 5050
+	1    0    0    -1
+$EndComp
+$Comp
+L CONN_01X14 P3
+U 1 1 5747820E
+P 9400 5050
+F 0 "P3" H 9400 5800 50  0000 C CNN
+F 1 "CONN_01X14" V 9500 5050 50  0000 C CNN
+F 2 "" H 9400 5050 50  0000 C CNN
+F 3 "" H 9400 5050 50  0000 C CNN
+	1    9400 5050
+	-1   0    0    -1
+$EndComp
+Text Notes 8950 5400 0    39   ~ 0
+Teensy 3.2\nconnection
+$Comp
+L CONN_01X03 P2
+U 1 1 57479630
+P 9300 4800
+F 0 "P2" H 9300 5000 50  0000 C CNN
+F 1 "CONN_01X03" V 9400 4800 50  0000 C CNN
+F 2 "" H 9300 4800 50  0000 C CNN
+F 3 "" H 9300 4800 50  0000 C CNN
+	1    9300 4800
+	1    0    0    -1
+$EndComp
+$Comp
+L CONN_01X05 P4
+U 1 1 57479992
+P 9100 5700
+F 0 "P4" V 9300 5700 50  0000 C CNN
+F 1 "CONN_01X05" V 9200 5700 50  0000 C CNN
+F 2 "" H 9100 5700 50  0000 C CNN
+F 3 "" H 9100 5700 50  0000 C CNN
+	1    9100 5700
+	0    -1   -1   0
+$EndComp
 $EndSCHEMATC
